File: layouts/default/default.kicad_pcb (KiCad board)
At the start: 2 copper layers, 156.5 x 33.5 mm, 17 parts

Commit message: Making sure everything is correct
Other:
- board text added: "Fabian Arévalo - 2025 Made with atopile"
Changed lines of the file:
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@@
 		(layer "Edge.Cuts")
+	)
+	(gr_text "Fabian Arévalo - 2025\nMade with atopile"
+		(at 230 105 0)
+		(layer "B.SilkS")
+		(effects
+			(font
+				(size 1.5 1.5)
+				(thickness 0.3)
+				(bold yes)
+			)
+			(justify left bottom mirror)
+		)
 	)
 	(via
